File: lego light controller.kicad_pcb (KiCad board)
At the start: 2 copper layers, 31.8 x 31.8 mm, 31 parts, among them J1 Conn_01x02, J2 Conn_01x02, J3 Conn_01x02, J4 Conn_01x03, J5 Conn_01x03, J7 Conn_01x06_Pin, P1 USB_C_Plug_USB2.0, Q1 BC847W, Q2 BC847W, Q3 BC847W, U1 ATSAMD11C14A-SS, U2 AMS1117-3.3

Commit message: add values and update usb c
Parts:
- removed R13, R14: R, Resistor_SMD:R_0402_1005Metric
- removed R3: R, Resistor_SMD:R_0603_1608Metric
- C1: value C_Polarized -> 10u
- C2: value C_Polarized -> 22u
- C3: value C -> 100n
- R1, R12, R2: value R -> 5k1
- R10, R11: value R -> 470
- R4, R5, R6: value R -> 10k
- R7, R8, R9: value R -> 1k
- moved R1 20.6 mm to (188.7, 81.5), turned to 90 degrees
- moved R2 18.4 mm to (186.5, 92.7), turned to -90 degrees
- moved Q3 3.48 mm to (204.0, 89.2), turned to 0 degrees
- moved R4 2.44 mm to (202.5, 86.3), turned to -90 degrees
- moved R9 2.26 mm to (201.0, 85.1), turned to 90 degrees
- moved R5 2.05 mm to (201.0, 88.2), turned to 90 degrees
- moved Q1 1.70 mm to (204.0, 94.5)
- moved Q2 1.70 mm to (204.0, 91.8)
- moved R6 1.70 mm to (201.5, 94.3)
- moved R7 1.40 mm to (201.2, 91.3)
- moved U2 1.10 mm to (195.7, 92.2)
- moved C2 0.90 mm to (189.3, 92.9)
- moved C1 0.40 mm to (182.8, 93.5)
- moved R12 0.40 mm to (192.2, 87.9)
Connections:
- P1 pad A5: unconnected-(P1-CC-PadA5) -> Net-(P1-CC1)
- P1 pad A6: /RUSB_P -> /USB_P
- P1 pad A7: /RUSB_N -> /USB_N
- P1 pad B5: unconnected-(P1-VCONN-PadB5) -> Net-(P1-CC2)
- P1 pad B6: (no net) -> /USB_P
- P1 pad B7: (no net) -> /USB_N
- Q1 pad 3: Net-(Q1-C) -> Net-(J3-Pin_2)
- Q2 pad 3: Net-(Q2-C) -> Net-(J2-Pin_2)
- Q3 pad 3: Net-(Q3-C) -> Net-(J1-Pin_2)
- R1 pad 1: Net-(Q1-C) -> Net-(P1-CC1)
- R1 pad 2: Net-(J3-Pin_2) -> GND
- R2 pad 1: Net-(Q2-C) -> Net-(P1-CC2)
- R2 pad 2: Net-(J2-Pin_2) -> GND
Routing:
- net Net-(P1-CC2): track 0.00 -> 9.22 mm, vias 0 -> 2
- net /USB_N: track 5.18 -> 12.6 mm
- net Net-(Q3-C): track 3.98 -> 0.00 mm
- net /USB_P: track 5.93 -> 9.55 mm
- net Net-(P1-CC1): track 0.00 -> 3.39 mm
- net /RUSB_N: track 3.35 -> 0.00 mm
- net /RUSB_P: track 3.11 -> 0.00 mm
- net /LED3: track 11.4 -> 13.8 mm
- net Net-(Q1-C): track 1.95 -> 0.00 mm
- net GND: track 4.17 -> 2.35 mm, vias 1 -> 7
- net Net-(Q2-C): track 1.66 -> 0.00 mm
- net Net-(Q3-B): track 5.03 -> 3.45 mm
- net /LED1: track 4.33 -> 5.91 mm
- net Net-(J7-Pin_3): track 3.95 -> 3.24 mm
- net Net-(Q2-B): track 7.33 -> 6.65 mm
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
Commit message: updates
Parts:
- added G***: LOGO, Custom:bee logo small, B.Cu at (190.5, 92.8)
Other:
- board text added: "YTvW 2024 LED controller Rev1.0"
- board text removed: "YTvW 2024 Lego LED controller Rev1.0"
