File: lego light controller.kicad_pcb (KiCad board)
At the start: 2 copper layers, 31.8 x 31.8 mm, 31 parts, among them J1 Conn_01x02, J2 Conn_01x02, J3 Conn_01x02, J4 Conn_01x03, J5 Conn_01x03, J7 Conn_01x06_Pin, P1 USB_C_Plug_USB2.0, Q1 BC847W, Q2 BC847W, Q3 BC847W, U1 ATSAMD11C14A-SS, U2 AP2111H-3.3TRG1

Commit message: fix pcb name
Other:
- board text added: "YTvW 2024 QBee LED controller Rev1.0"
- board text removed: "YTvW 2024 LED controller Rev1.0"
Changed lines of the file:
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@@
 	)
 	(paper "A4")
+	(title_block
+		(comment 4 "AISLER Project ID: AIXNFFQP")
+	)
 	(layers
 		(0 "F.Cu" signal)
@@
 		(tags "Capacitor Electrolytic")
 		(property "Reference" "C1"
-			(at -0.96 -0.2 90)
+			(at -0.96 -1.17 90)
 			(layer "B.SilkS")
 			(effects
@@
 		)
 	)
-	(gr_text "YTvW 2024 \nLED controller\nRev1.0"
+	(gr_text "YTvW 2024 \nQBee LED controller\nRev1.0"
 		(at 190.38 80.06 90)
 		(layer "B.SilkS")

Commit message: small fixes
Routing:
- net +5V: track 73.0 -> 74.2 mm
