File: lego light controller.kicad_pcb (KiCad board)
At the start: 2 copper layers, 31.8 x 31.8 mm, 31 parts, among them J1 Conn_01x02, J2 Conn_01x02, J3 Conn_01x02, J4 Conn_01x03, J5 Conn_01x03, J7 Conn_01x06_Pin, P1 USB_C_Plug_USB2.0, Q1 BC847W, Q2 BC847W, Q3 BC847W, U1 ATSAMD11C14A-SS, U2 AP2111H-3.3TRG1

Commit message: start working on hardware revision 2
Parts:
- added J6: Conn_01x03, Connector_PinHeader_2.54mm:PinHeader_1x03_P2.54mm_Vertical, F.Cu at (205.1, 84.6)
- added Q4: BC847W, Package_TO_SOT_SMD:SOT-23, F.Cu at (218.2, 94.2)
- added R13: 5k1, Resistor_SMD:R_0603_1608Metric, F.Cu at (185.9, 67.5)
- added R3: 10k, Resistor_SMD:R_0603_1608Metric, F.Cu at (201.2, 91.5)
- added U3: ATSAMD21E17D-A, Package_QFP:TQFP-32_7x7mm_P0.8mm, B.Cu at (198.5, 88.1)
- added U4: SN74LVC1T45DCK, Package_TO_SOT_SMD:SOT-363_SC-70-6, F.Cu at (200.7, 85.1)
- C3: moved to B.Cu
- J4: value Conn_01x03 -> Conn_01x02; footprint Connector_PinHeader_2.54mm:PinHeader_1x03_P2.54mm_Vertical -> Connector_PinHeader_2.54mm:PinHeader_1x02_P2.54mm_Vertical
- R1, R2: value 5k1 -> 1k; moved to F.Cu
- R11: value 470 -> 5k1; moved to B.Cu
- R5, R6: value 10k -> 1k
- R7, R8: value 1k -> 10k
- R9: value 1k -> 470
- U1: value ATSAMD11C14A-SS -> AP2111H-3.3TRG1; footprint Package_SO:SOIC-14_3.9x8.7mm_P1.27mm -> Package_TO_SOT_SMD:SOT-223-3_TabPin2
- U2: value AP2111H-3.3TRG1 -> SN74LVC1T45DCK; footprint Package_TO_SOT_SMD:SOT-223-3_TabPin2 -> Package_TO_SOT_SMD:SOT-363_SC-70-6
- moved TP2 25.2 mm to (179.4, 107.4)
- moved R11 20.7 mm to (182.2, 84.4), turned to 180 degrees
- moved TP1 19.5 mm to (183.4, 107.4)
- moved J7 17.3 mm to (192.9, 66.5)
- moved R1 15.7 mm to (197.6, 86.9)
- moved R2 13.7 mm to (195.8, 90.9), turned to 90 degrees
- moved R12 12.7 mm to (182.2, 92.9), turned to 180 degrees
- moved J4 12.1 mm to (210.0, 95.8), turned to -90 degrees
- moved U2 10.4 mm to (200.7, 81.5), turned to 90 degrees
- moved R9 9.26 mm to (202.6, 81.5)
- moved C3 8.24 mm to (193.5, 82.3), turned to -135 degrees
- moved R4 8.21 mm to (196.4, 88.6)
- moved Q2 7.46 mm to (203.8, 91.4)
- moved U1 7.41 mm to (190.8, 84.5), turned to -90 degrees
- moved Q1 5.92 mm to (203.8, 88.1)
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Connections:
- J7 pad 2: Net-(J7-Pin_2) -> /~{RST}
- J7 pad 3: Net-(J7-Pin_3) -> /SWCLK
- J7 pad 4: Net-(J7-Pin_4) -> /SWDIO
- Q1 pad 3: Net-(J3-Pin_2) -> Net-(J1-Pin_2)
- Q3 pad 3: Net-(J1-Pin_2) -> Net-(J3-Pin_2)
- R1 pad 1: Net-(P1-CC1) -> Net-(Q1-B)
- R1 pad 2: GND -> /LED1
- R10 pad 1: Net-(J4-Pin_2) -> Net-(J6-Pin_2)
- R10 pad 2: /DL1 -> Net-(U4-B)
- R11 pad 1: Net-(J5-Pin_2) -> Net-(P1-CC1)
- R11 pad 2: /DL2 -> GND
- R12 pad 1: +3V3 -> Net-(P1-CC2)
- R12 pad 2: Net-(J7-Pin_2) -> GND
- R2 pad 1: Net-(P1-CC2) -> Net-(Q2-B)
- R2 pad 2: GND -> /LED2
- R4 pad 2: Net-(Q3-B) -> Net-(Q2-B)
- R5 pad 1: GND -> Net-(Q3-B)
- R5 pad 2: Net-(Q2-B) -> /LED3
- R6 pad 1: GND -> Net-(Q4-B)
- R6 pad 2: Net-(Q1-B) -> /LED4
- R7 pad 1: Net-(Q1-B) -> GND
- R7 pad 2: /LED3 -> Net-(Q3-B)
- R8 pad 1: Net-(Q2-B) -> GND
- R8 pad 2: /LED2 -> Net-(Q4-B)
- R9 pad 1: Net-(Q3-B) -> Net-(J5-Pin_2)
- R9 pad 2: /LED1 -> Net-(U2-B)
- U1 pad 1: /LED3 -> GND
- U1 pad 2: /EXT1 -> +3V3
- U1 pad 3: /EXT2 -> +5V
- U2 pad 1: GND -> +3V3
- U2 pad 2: +3V3 -> GND
- U2 pad 3: +5V -> /DL1
Routing:
- net +3V3: track 24.0 -> 0.00 mm, vias 2 -> 0
- net Net-(J2-Pin_2): track 11.5 -> 0.00 mm
- net /LED3: track 9.89 -> 0.00 mm, vias 2 -> 0
- net Net-(J7-Pin_2): track 9.44 -> 0.00 mm, vias 1 -> 0
- net /EXT1: track 9.35 -> 0.00 mm, vias 1 -> 0
- net /EXT2: track 7.27 -> 0.00 mm, vias 1 -> 0
- net /LED1: track 7.05 -> 0.00 mm
- net Net-(Q2-B): track 6.33 -> 0.00 mm
- net Net-(J7-Pin_3): track 6.17 -> 0.00 mm, vias 1 -> 0
- net Net-(J4-Pin_2): track 5.96 -> 0.00 mm
- net Net-(J5-Pin_2): track 5.86 -> 0.00 mm
- net Net-(J7-Pin_4): track 4.97 -> 0.00 mm, vias 1 -> 0
- net Net-(J1-Pin_2): track 3.75 -> 0.00 mm
- net Net-(Q3-B): track 3.64 -> 0.00 mm
- net /LED2: track 3.41 -> 0.00 mm
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