File: lego light controller.kicad_sch (KiCad schematic)
At the start: 30 parts, among them J1 Conn_01x02, J2 Conn_01x02, J3 Conn_01x02, J4 Conn_01x03, J5 Conn_01x03, J7 Conn_01x06_Pin, P1 USB_C_Plug_USB2.0, Q1 BC847W, Q2 BC847W, Q3 BC847W, U1 ATSAMD11C14A-SS, U2 AP2111H-3.3TRG1

Commit message: fix BOM
Parts:
- H1, H2: now not fitted; now left out of the parts list
Changed lines of the file:
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@@
 		(unit 1)
 		(exclude_from_sim no)
-		(in_bom yes)
-		(on_board yes)
-		(dnp no)
+		(in_bom no)
+		(on_board yes)
+		(dnp yes)
 		(fields_autoplaced yes)
 		(property "Reference" "H1"
@@
 		(unit 1)
 		(exclude_from_sim no)
-		(in_bom yes)
-		(on_board yes)
-		(dnp no)
+		(in_bom no)
+		(on_board yes)
+		(dnp yes)
 		(fields_autoplaced yes)
 		(property "Reference" "H2"
