File: lego light controller.kicad_sch (KiCad schematic)
At the start: 30 parts, among them J1 Conn_01x02, J2 Conn_01x02, J3 Conn_01x02, J4 Conn_01x03, J5 Conn_01x03, J7 Conn_01x06_Pin, P1 USB_C_Plug_USB2.0, Q1 BC847W, Q2 BC847W, Q3 BC847W, U1 ATSAMD11C14A-SS, U2 AP2111H-3.3TRG1

Commit message: start working on hardware revision 2
Parts:
- removed R9: 1k, Resistor_SMD:R_0603_1608Metric, symbol Device:R
- removed U1: ATSAMD11C14A-SS, Package_SO:SOIC-14_3.9x8.7mm_P1.27mm, symbol MCU_Microchip_SAMD:ATSAMD11C14A-SS
- added J4: Conn_01x02, Connector_PinHeader_2.54mm:PinHeader_1x02_P2.54mm_Vertical, symbol Connector_Generic:Conn_01x02
- added Q4: BC847W, Package_TO_SOT_SMD:SOT-23, symbol Transistor_BJT:BC847W
- added R1, R2: 1k, Resistor_SMD:R_0603_1608Metric, symbol Device:R
- added R3: 10k, Resistor_SMD:R_0603_1608Metric, symbol Device:R
- added U2, U4: SN74LVC1T45DCK, Package_TO_SOT_SMD:SOT-363_SC-70-6, symbol Logic_LevelTranslator:SN74LVC1T45DCK
- added U3: ATSAMD21E17D-A, Package_QFP:TQFP-32_7x7mm_P0.8mm, symbol MCU_Microchip_SAMD:ATSAMD21E17D-A
- R5, R6: value 10k -> 1k
- R7, R8: value 1k -> 10k
- renumbered J4 to J5, J5 to J6, R11 to R10, R1 to R11, R2 to R12, R12 to R13, R10 to R9, U2 to U1
Connections:
- net +3V3: now also U2.1 (VCCA), U2.5 (DIR), U3.30 (VDDIN), U4.1 (VCCA), U4.5 (DIR)
- net +5V: now also J4.1 (Pin_1), U2.6 (VCCB), U4.6 (VCCB)
- net DL1: now also U2.3 (A), U3.5 (PA04); no longer R9.2
- net DL2: now also U3.6 (PA05); no longer R10.2
- net GND: now also R7.1, R8.1, Q4.2 (E), R3.1, U2.2 (GND), U4.2 (GND); no longer R5.1, R6.1
- net LED1: now also R1.2, U3.15 (PA14)
- net LED2: now also R2.2, U3.16 (PA15); no longer R8.2
- net LED3: now also R5.2, U3.21 (PA22); no longer R7.2
- net USB_N: now also U3.23 (PA24)
- net USB_P: now also U3.24 (PA25)
- net at Q1.3 (C): now also J1.2 (Pin_2); no longer J3.2 (Pin_2)
- net ~{RST}: now reaches J7.2 (Pin_2), R13.2
- net ~{RST}: now also U3.26 (~{RESET})
- net SWCLK: now reaches J7.3 (Pin_3)
- net SWCLK: now also U3.31 (PA30)
- net SWDIO: now reaches J7.4 (Pin_4)
- net SWDIO: now also U3.32 (PA31)
- net at Q3.3 (C): now also J3.2 (Pin_2); no longer J1.2 (Pin_2)
- net at Q3.1 (B): now also R5.1, R7.2; no longer R4.2
- new net: Q1.1 (B), R1.1, R3.2
- new net: J4.2 (Pin_2), Q4.3 (C)
- new net: U3.10 (GND), U3.28 (GND)
- new net: R9.2, U2.4 (B)
- new net: R10.2, U4.4 (B)
- new net: Q4.1 (B), R6.1, R8.2
- new net: Q2.1 (B), R2.1, R4.2
- new net LED4: R6.2, U3.22 (PA23)
Other:
- note added: "PWM leds"
- note removed: "Pwm Leds"
- moved on the sheet: C3, H1, H2, J5, J6, J7, P1, R10, R11, R12, R13, R9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
